File: pcb/barn_door/barn_door.sch (KiCad schematic (older format))
At the start: 26 parts, among them J1 MOTOR_OUT, J2 HEATER, Q1 Q_NMOS_DGS, SW1 REVERSE, SW2 ENDSTOP, SW3 START, U1 HEATER_TEMP, U2 OUTDOOR_TEMP, U3 LM358, U4 bluepill

Commit message: Fix diff amp
Connections:
- net GND: now also R10.1, R9.1; no longer R7.2, R8.2
- net TEMP_HEATER: now also R7.2; no longer R9.1
- net TEMP_OUTDOOR: now also R8.2; no longer R10.1
Changed lines of the file:
@@
 	0    -1   -1   0
-$EndComp
-$Comp
-L Device:R R8
-U 1 1 5EC66A6D
-P 2700 2050
-F 0 "R8" H 2770 2096 50  0000 L CNN
-F 1 "R" H 2770 2005 50  0000 L CNN
-F 2 "" V 2630 2050 50  0001 C CNN
-F 3 "~" H 2700 2050 50  0001 C CNN
-	1    2700 2050
-	1    0    0    -1
 $EndComp
 Wire Wire Line
@@
 Wire Wire Line
 	2700 1850 2850 1850
-$Comp
-L power:GND #PWR08
-U 1 1 5EC699E3
-P 2700 2200
-F 0 "#PWR08" H 2700 1950 50  0001 C CNN
-F 1 "GND" H 2705 2027 50  0000 C CNN
-F 2 "" H 2700 2200 50  0001 C CNN
-F 3 "" H 2700 2200 50  0001 C CNN
-	1    2700 2200
-	1    0    0    -1
-$EndComp
 Wire Wire Line
 	2850 1650 2750 1650
 Wire Wire Line
 	2400 1650 2400 1500
-$Comp
-L Device:R R10
-U 1 1 5EC6ABBB
-P 2750 1350
-F 0 "R10" H 2820 1396 50  0000 L CNN
-F 1 "R" H 2820 1305 50  0000 L CNN
-F 2 "" V 2680 1350 50  0001 C CNN
-F 3 "~" H 2750 1350 50  0001 C CNN
-	1    2750 1350
-	1    0    0    -1
-$EndComp
 Wire Wire Line
 	2750 1650 2750 1500
@@
 Wire Wire Line
 	2750 1650 2400 1650
-Wire Wire Line
-	2750 1200 3450 1200
-Wire Wire Line
-	3450 1200 3450 1750
 Text Label 4100 1750 2    50   ~ 0
 TEMP_OUTDOOR
-Connection ~ 3450 1750
-Wire Wire Line
-	3450 1750 4100 1750
+Wire Wire Line
+	3450 1750 3500 1750
 $Comp
 L Sensor_Temperature:LM35-LP U1
@@
 L power:GND #PWR07
 U 1 1 5EC71C26
-P 2650 4400
-F 0 "#PWR07" H 2650 4150 50  0001 C CNN
-F 1 "GND" H 2655 4227 50  0000 C CNN
-F 2 "" H 2650 4400 50  0001 C CNN
-F 3 "" H 2650 4400 50  0001 C CNN
-	1    2650 4400
-	1    0    0    -1
+P 2700 3400
+F 0 "#PWR07" H 2700 3150 50  0001 C CNN
+F 1 "GND" H 2705 3227 50  0000 C CNN
+F 2 "" H 2700 3400 50  0001 C CNN
+F 3 "" H 2700 3400 50  0001 C CNN
+	1    2700 3400
+	-1   0    0    1
 $EndComp
 Wire Wire Line
@@
 Wire Wire Line
 	2700 3850 2350 3850
-Wire Wire Line
-	2700 3400 3400 3400
-Wire Wire Line
-	3400 3400 3400 3950
 Text Label 3950 3950 2    50   ~ 0
 TEMP_HEATER
 Wire Wire Line
-	3400 3950 3950 3950
-Connection ~ 3400 3950
+	3400 3950 3450 3950
 $Comp
 L my_components:bluepill U4
@@
 Wire Wire Line
 	5950 1950 6350 1950
+$Comp
+L Device:R R10
+U 1 1 5EC6ABBB
+P 2750 1350
+F 0 "R10" H 2820 1396 50  0000 L CNN
+F 1 "R" H 2820 1305 50  0000 L CNN
+F 2 "" V 2680 1350 50  0001 C CNN
+F 3 "~" H 2750 1350 50  0001 C CNN
+	1    2750 1350
+	1    0    0    -1
+$EndComp
+$Comp
+L power:GND #PWR08
+U 1 1 5EC699E3
+P 2750 1200
+F 0 "#PWR08" H 2750 950 50  0001 C CNN
+F 1 "GND" H 2755 1027 50  0000 C CNN
+F 2 "" H 2750 1200 50  0001 C CNN
+F 3 "" H 2750 1200 50  0001 C CNN
+	1    2750 1200
+	-1   0    0    1
+$EndComp
+$Comp
+L Device:R R8
+U 1 1 5EC66A6D
+P 2700 2050
+F 0 "R8" H 2770 2096 50  0000 L CNN
+F 1 "R" H 2770 2005 50  0000 L CNN
+F 2 "" V 2630 2050 50  0001 C CNN
+F 3 "~" H 2700 2050 50  0001 C CNN
+	1    2700 2050
+	1    0    0    -1
+$EndComp
+Wire Wire Line
+	2700 2200 3500 2200
+Wire Wire Line
+	3500 2200 3500 1750
+Connection ~ 3500 1750
+Wire Wire Line
+	3500 1750 4100 1750
+Wire Wire Line
+	2650 4400 3450 4400
+Wire Wire Line
+	3450 4400 3450 3950
+Connection ~ 3450 3950
+Wire Wire Line
+	3450 3950 3950 3950
 $EndSCHEMATC

Commit message: Really fix the op amp. I was just stupid :/
Parts:
- removed D1, D2: D, symbol Device:D
- removed R10, R9: R, symbol Device:R
- R4, R6: value R -> 10k
- R7, R8: value R -> 100k
Connections:
- net +3V3: no longer U1.1 (+VS), U2.1 (+VS)
- net +5V: now also U1.1 (+VS), U2.1 (+VS)
- net GND: now also R4.1, R6.1
- net TEMP_GND: now reaches D3.2 (A), U2.3 (GND)
- net TEMP_GND: now also U1.3 (GND); no longer R6.1
Other:
- moved on the sheet: D3, D4
Changed lines of the file:
@@
 L Device:D D3
 U 1 1 5EC518CE
-P 1500 2050
-F 0 "D3" V 1546 1970 50  0000 R CNN
-F 1 "D" V 1455 1970 50  0000 R CNN
-F 2 "" H 1500 2050 50  0001 C CNN
-F 3 "~" H 1500 2050 50  0001 C CNN
-	1    1500 2050
+P 800 2650
+F 0 "D3" V 846 2570 50  0000 R CNN
+F 1 "D" V 755 2570 50  0000 R CNN
+F 2 "" H 800 2650 50  0001 C CNN
+F 3 "~" H 800 2650 50  0001 C CNN
+	1    800  2650
 	0    -1   -1   0
 $EndComp
@@
 L Device:D D4
 U 1 1 5EC521FA
-P 1500 2400
-F 0 "D4" V 1546 2320 50  0000 R CNN
-F 1 "D" V 1455 2320 50  0000 R CNN
-F 2 "" H 1500 2400 50  0001 C CNN
-F 3 "~" H 1500 2400 50  0001 C CNN
-	1    1500 2400
-	0    -1   -1   0
-$EndComp
-Wire Wire Line
-	1500 2250 1500 2200
+P 800 3000
+F 0 "D4" V 846 2920 50  0000 R CNN
+F 1 "D" V 755 2920 50  0000 R CNN
+F 2 "" H 800 3000 50  0001 C CNN
+F 3 "~" H 800 3000 50  0001 C CNN
+	1    800  3000
+	0    -1   -1   0
+$EndComp
+Wire Wire Line
+	800  2850 800  2800
 $Comp
 L power:GND #PWR04
 U 1 1 5EC52858
-P 1500 2550
-F 0 "#PWR04" H 1500 2300 50  0001 C CNN
-F 1 "GND" H 1505 2377 50  0000 C CNN
-F 2 "" H 1500 2550 50  0001 C CNN
-F 3 "" H 1500 2550 50  0001 C CNN
-	1    1500 2550
-	1    0    0    -1
-$EndComp
-$Comp
-L power:+3.3V #PWR03
-U 1 1 5EC53415
-P 1500 1050
-F 0 "#PWR03" H 1500 900 50  0001 C CNN
-F 1 "+3.3V" H 1515 1223 50  0000 C CNN
-F 2 "" H 1500 1050 50  0001 C CNN
-F 3 "" H 1500 1050 50  0001 C CNN
-	1    1500 1050
+P 800 3150
+F 0 "#PWR04" H 800 2900 50  0001 C CNN
+F 1 "GND" H 805 2977 50  0000 C CNN
+F 2 "" H 800 3150 50  0001 C CNN
+F 3 "" H 800 3150 50  0001 C CNN
+	1    800  3150
 	1    0    0    -1
 $EndComp
@@
 P 2250 1850
 F 0 "R6" V 2457 1850 50  0000 C CNN
-F 1 "R" V 2366 1850 50  0000 C CNN
+F 1 "10k" V 2250 1850 50  0000 C CNN
 F 2 "" V 2180 1850 50  0001 C CNN
 F 3 "~" H 2250 1850 50  0001 C CNN
@@
 	2700 1850 2850 1850
 Wire Wire Line
-	2850 1650 2750 1650
-Wire Wire Line
 	2400 1650 2400 1500
-Wire Wire Line
-	2750 1650 2750 1500
-Connection ~ 2750 1650
-Wire Wire Line
-	2750 1650 2400 1650
 Text Label 4100 1750 2    50   ~ 0
 TEMP_OUTDOOR
@@
 F 3 "http://www.ti.com/lit/ds/symlink/lm35.pdf" H 1450 3700 50  0001 C CNN
 	1    1450 3700
-	1    0    0    -1
-$EndComp
-$Comp
-L Device:D D1
-U 1 1 5EC71BB5
-P 1450 4250
-F 0 "D1" V 1496 4170 50  0000 R CNN
-F 1 "D" V 1405 4170 50  0000 R CNN
-F 2 "" H 1450 4250 50  0001 C CNN
-F 3 "~" H 1450 4250 50  0001 C CNN
-	1    1450 4250
-	0    -1   -1   0
-$EndComp
-$Comp
-L Device:D D2
-U 1 1 5EC71BBF
-P 1450 4600
-F 0 "D2" V 1496 4520 50  0000 R CNN
-F 1 "D" V 1405 4520 50  0000 R CNN
-F 2 "" H 1450 4600 50  0001 C CNN
-F 3 "~" H 1450 4600 50  0001 C CNN
-	1    1450 4600
-	0    -1   -1   0
-$EndComp
-Wire Wire Line
-	1450 4450 1450 4400
-$Comp
-L power:GND #PWR02
-U 1 1 5EC71BCB
-P 1450 4750
-F 0 "#PWR02" H 1450 4500 50  0001 C CNN
-F 1 "GND" H 1455 4577 50  0000 C CNN
-F 2 "" H 1450 4750 50  0001 C CNN
-F 3 "" H 1450 4750 50  0001 C CNN
-	1    1450 4750
-	1    0    0    -1
-$EndComp
-$Comp
-L power:+3.3V #PWR01
-U 1 1 5EC71BD5
-P 1450 3250
-F 0 "#PWR01" H 1450 3100 50  0001 C CNN
-F 1 "+3.3V" H 1465 3423 50  0000 C CNN
-F 2 "" H 1450 3250 50  0001 C CNN
-F 3 "" H 1450 3250 50  0001 C CNN
-	1    1450 3250
 	1    0    0    -1
 $EndComp
@@
 P 2200 4050
 F 0 "R4" V 2407 4050 50  0000 C CNN
-F 1 "R" V 2316 4050 50  0000 C CNN
+F 1 "10k" V 2200 4050 50  0000 C CNN
 F 2 "" V 2130 4050 50  0001 C CNN
 F 3 "~" H 2200 4050 50  0001 C CNN
@@
 P 2650 4250
 F 0 "R7" H 2720 4296 50  0000 L CNN
-F 1 "R" H 2720 4205 50  0000 L CNN
+F 1 "100k" V 2650 4150 50  0000 L CNN
 F 2 "" V 2580 4250 50  0001 C CNN
 F 3 "~" H 2650 4250 50  0001 C CNN
@@
 Wire Wire Line
 	2650 4050 2800 4050
-$Comp
-L power:GND #PWR07
-U 1 1 5EC71C26
-P 2700 3400
-F 0 "#PWR07" H 2700 3150 50  0001 C CNN
-F 1 "GND" H 2705 3227 50  0000 C CNN
-F 2 "" H 2700 3400 50  0001 C CNN
-F 3 "" H 2700 3400 50  0001 C CNN
-	1    2700 3400
-	-1   0    0    1
-$EndComp
-Wire Wire Line
-	2800 3850 2700 3850
 Wire Wire Line
 	2350 3850 2350 3700
-$Comp
-L Device:R R9
-U 1 1 5EC71C33
-P 2700 3550
-F 0 "R9" H 2770 3596 50  0000 L CNN
-F 1 "R" H 2770 3505 50  0000 L CNN
-F 2 "" V 2630 3550 50  0001 C CNN
-F 3 "~" H 2700 3550 50  0001 C CNN
-	1    2700 3550
-	1    0    0    -1
-$EndComp
-Wire Wire Line
-	2700 3850 2700 3700
-Connection ~ 2700 3850
-Wire Wire Line
-	2700 3850 2350 3850
 Text Label 3950 3950 2    50   ~ 0
 TEMP_HEATER
@@
 $EndComp
 Wire Wire Line
-	1500 1800 1500 1850
-Wire Wire Line
-	2100 1850 1500 1850
-Connection ~ 1500 1850
-Wire Wire Line
-	1500 1850 1500 1900
-Wire Wire Line
 	2100 1500 2050 1500
 Connection ~ 2050 1500
 Wire Wire Line
-	1450 4000 1450 4050
-Wire Wire Line
 	2050 3700 2000 3700
 Connection ~ 2000 3700
-Wire Wire Line
-	2050 4050 1450 4050
-Connection ~ 1450 4050
-Wire Wire Line
-	1450 4050 1450 4100
 Wire Notes Line
 	450  5150 4400 5150
@@
 	5950 1950 6350 1950
 $Comp
-L Device:R R10
-U 1 1 5EC6ABBB
-P 2750 1350
-F 0 "R10" H 2820 1396 50  0000 L CNN
-F 1 "R" H 2820 1305 50  0000 L CNN
-F 2 "" V 2680 1350 50  0001 C CNN
-F 3 "~" H 2750 1350 50  0001 C CNN
-	1    2750 1350
-	1    0    0    -1
-$EndComp
-$Comp
-L power:GND #PWR08
-U 1 1 5EC699E3
-P 2750 1200
-F 0 "#PWR08" H 2750 950 50  0001 C CNN
-F 1 "GND" H 2755 1027 50  0000 C CNN
-F 2 "" H 2750 1200 50  0001 C CNN
-F 3 "" H 2750 1200 50  0001 C CNN
-	1    2750 1200
-	-1   0    0    1
-$EndComp
-$Comp
 L Device:R R8
 U 1 1 5EC66A6D
 P 2700 2050
 F 0 "R8" H 2770 2096 50  0000 L CNN
-F 1 "R" H 2770 2005 50  0000 L CNN
+F 1 "100k" V 2700 1950 50  0000 L CNN
 F 2 "" V 2630 2050 50  0001 C CNN
 F 3 "~" H 2700 2050 50  0001 C CNN
@@
 Wire Wire Line
 	3450 3950 3950 3950
+Text Label 800  2100 3    50   ~ 0
+TEMP_GND
+Wire Wire Line
+	800  2500 800  2100
+Text Label 1500 2300 1    50   ~ 0
+TEMP_GND
+Text Label 1450 4500 1    50   ~ 0
+TEMP_GND
+$Comp
+L power:+5V #PWR?
+U 1 1 5EC7FA83
+P 1450 3250
+F 0 "#PWR?" H 1450 3100 50  0001 C CNN
+F 1 "+5V" V 1465 3378 50  0000 L CNN
+F 2 "" H 1450 3250 50  0001 C CNN
+F 3 "" H 1450 3250 50  0001 C CNN
+	1    1450 3250
+	1    0    0    -1
+$EndComp
+$Comp
+L power:+5V #PWR?
+U 1 1 5EC80300
+P 1500 1050
+F 0 "#PWR?" H 1500 900 50  0001 C CNN
+F 1 "+5V" V 1515 1178 50  0000 L CNN
+F 2 "" H 1500 1050 50  0001 C CNN
+F 3 "" H 1500 1050 50  0001 C CNN
+	1    1500 1050
+	1    0    0    -1
+$EndComp
+Wire Wire Line
+	2350 3850 2800 3850
+Wire Wire Line
+	1450 4000 1450 4500
+$Comp
+L power:GND #PWR?
+U 1 1 5EC66C7A
+P 2050 4200
+F 0 "#PWR?" H 2050 3950 50  0001 C CNN
+F 1 "GND" H 2055 4027 50  0000 C CNN
+F 2 "" H 2050 4200 50  0001 C CNN
+F 3 "" H 2050 4200 50  0001 C CNN
+	1    2050 4200
+	1    0    0    -1
+$EndComp
+Wire Wire Line
+	2050 4050 2050 4200
+Wire Wire Line
+	2400 1650 2850 1650
+Wire Wire Line
+	1500 1800 1500 2300
+$Comp
+L power:GND #PWR?
+U 1 1 5EC68B16
+P 2050 1950
+F 0 "#PWR?" H 2050 1700 50  0001 C CNN
+F 1 "GND" H 2055 1777 50  0000 C CNN
+F 2 "" H 2050 1950 50  0001 C CNN
+F 3 "" H 2050 1950 50  0001 C CNN
+	1    2050 1950
+	1    0    0    -1
+$EndComp
+Wire Wire Line
+	2050 1950 2050 1850
+Wire Wire Line
+	2050 1850 2100 1850
 $EndSCHEMATC
